File: Hardware/MeteoNode.kicad_sch (KiCad schematic)
At the start: 22 parts, among them J1 HTU21D_Module, J2 BMP280_Module, J3 TP5000_Charge_Module, J4 2W_5V_Solar_Panel, J5 32700_LiFePO4_Battery, J6 2W_5V_Solar_Panel, Q1 FDN304P, Q2 2N7000, SW1 Momentary, U1 ESP32-WROOM-32UE

Commit message: add Updated schematic
Parts:
- R1, R2: value R -> 100kΩ
Changed lines of the file:
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@@
       (effects (font (size 1.27 1.27)) (justify left))
     )
-    (property "Value" "R" (id 1) (at 99.06 124.4599 0)
+    (property "Value" "100kΩ" (id 1) (at 99.06 124.4599 0)
       (effects (font (size 1.27 1.27)) (justify left))
     )
@@
       (effects (font (size 1.27 1.27)) (justify left))
     )
-    (property "Value" "R" (id 1) (at 99.06 134.6199 0)
+    (property "Value" "100kΩ" (id 1) (at 99.06 134.6199 0)
       (effects (font (size 1.27 1.27)) (justify left))
     )
@@
     )
     (path "/3e50bec7-8765-4cb4-8a85-464ed97b18bf"
-      (reference "R1") (unit 1) (value "R") (footprint "")
+      (reference "R1") (unit 1) (value "100kΩ") (footprint "")
     )
     (path "/5a7b5f42-23ed-440e-9fd0-33baa29da793"
-      (reference "R2") (unit 1) (value "R") (footprint "")
+      (reference "R2") (unit 1) (value "100kΩ") (footprint "")
     )
     (path "/f89b44fd-1fe0-4315-acaa-6aedbac4e8d4"
